File: Hardware/esp01-ws2812b-breakout/esp01-ws2812b-breakout.sch (KiCad schematic (older format))
At the start: 11 parts, among them J1 Screw_Terminal_01x02, J2 Screw_Terminal_01x04, U1 LM1117-3.3, U2 DS18B20, U3 ESP-01v090

Commit message: Included level shifters for LED data pins
Parts:
- removed R1, R2: 470, symbol Device:R
- added 10k (x2), 10k? (x2): R, symbol Device:R
- added Q? (x2): IRFS4127, Package_TO_SOT_SMD:TO-263-2, symbol Transistor_FET:IRFS4127
Connections:
- net +3V3: now also 10k.1, 10k?.1, Q?.1 (G), Q?.1 (G)
- net +5V: now also 10k.1, 10k?.1
- net LED1_5V: now reaches J2.2 (Pin_2)
- net LED1_5V: now also 10k.2, Q?.2 (D)
- net LED2_5V: now reaches J2.3 (Pin_3)
- net LED2_5V: now also 10k?.2, Q?.2 (D)
- net LED1 renamed LED1_3V3
- net LED1_3V3: now also 10k.2, Q?.3 (S)
- net LED2 renamed LED2_3V3
- net LED2_3V3: now also 10k?.2, Q?.3 (S)
Other:
- note added: "Level shifter for LED data pin 1 and 2 \nBased on: https://www.nxp.com/docs/en/application-note/AN10441.pdf"
- moved on the sheet: 10uF1, 10uF2, C1, J2, R3, U1, U2

Commit message: Schematics completed, PCB design started
Parts:
- added J3: Conn_01x03_Male, Connector_PinHeader_2.54mm:PinHeader_1x03_P2.54mm_Vertical, symbol Connector:Conn_01x03_Male
- added R5: 10K, Resistor_SMD:R_0603_1608Metric_Pad0.98x0.95mm_HandSolder, symbol Device:R
- C1: renamed from 10uF1; value C -> 10uF; footprint (none) -> Capacitor_SMD:C_0603_1608Metric_Pad1.08x0.95mm_HandSolder
- C2: renamed from 10uF2; value C -> 10uF; footprint (none) -> Capacitor_SMD:C_0603_1608Metric_Pad1.08x0.95mm_HandSolder
- C3: renamed from C1; footprint (none) -> Capacitor_SMD:C_0603_1608Metric_Pad1.08x0.95mm_HandSolder
- J1: footprint (none) -> Connector_PinHeader_2.54mm:PinHeader_1x04_P2.54mm_Vertical
- J2: footprint (none) -> Connector_PinHeader_2.54mm:PinHeader_1x08_P2.54mm_Vertical
- Q1, Q2: renamed from Q?; footprint Package_TO_SOT_SMD:TO-263-2 -> ESP8266:SOT-23_Handsoldering_DS-REVERSED
- R1, R2: renamed from 10k; value R -> 10K; footprint (none) -> Resistor_SMD:R_0603_1608Metric_Pad0.98x0.95mm_HandSolder
- R3, R4: renamed from 10k?; value R -> 10K; footprint (none) -> Resistor_SMD:R_0603_1608Metric_Pad0.98x0.95mm_HandSolder
- R6: renamed from R3; value 4.7K -> 4K7; footprint (none) -> Resistor_SMD:R_0603_1608Metric_Pad0.98x0.95mm_HandSolder
- U1: footprint (none) -> Package_TO_SOT_SMD:SOT-223
- U2: renamed from U3; footprint (none) -> ESP8266:ESP-01
- renumbered U2 to U3
Connections:
- net +3V3: now also J3.2 (Pin_2), J3.3 (Pin_3), R5.2
- net GND: now also J3.1 (Pin_1)
- net GPIO0: now reaches U2.6 (GPIO0)
- net GPIO0: now also R5.1
- no-connect marks 2 -> 1
Other:
- note added: "(Optional) interface to interact with GPIO0\n10k pullup ensures the ESP01 boots in correct mode"
- note added: "DS18B20 temperature sensor"
- note added: "ESP-01 MCU"
- note added: "LED connection terminal"
- note removed: "MCU Unit"
- moved on the sheet: C3, J1, J2, R6, U2, U3
